Commit message: feat(urdf): improved arm urdf and add STL align to CoM - added STL align to CoM - renamed links that starting from zero not to one like DH convention - fixed gripper with correct STLs position

File: open_manipulator_x_description/gazebo/open_manipulator_x.gazebo.xacro (robot description, xacro)
@@ -29,9 +29,9 @@
     </gazebo>
   </xacro:macro>
+  <xacro:Link reference="${prefix}link0"/>
   <xacro:Link reference="${prefix}link1"/>
   <xacro:Link reference="${prefix}link2"/>
   <xacro:Link reference="${prefix}link3"/>
   <xacro:Link reference="${prefix}link4"/>
-  <xacro:Link reference="${prefix}link5"/>
   <xacro:Link reference="${prefix}gripper_left_link"/>
   <xacro:Link reference="${prefix}gripper_right_link"/>

File: open_manipulator_x_description/urdf/open_manipulator_x.urdf.xacro (robot description, xacro)
@@ -6,175 +6,178 @@
       name="meshes_file_direction"
       value="package://open_manipulator_x_description/meshes"/>
+    <xacro:property name="CoM_link0" value="${[2.0, 0.0, 0.0]}" />
+    <link name="${prefix}link0">
+      <visual>
+        <origin xyz="0.0011 -0.0001 0.0194" rpy="0 0 0"/>
+        <geometry>
+          <mesh filename="${meshes_file_direction}/pieces_CoM/link0_CoM.stl" scale="0.001 0.001 0.001"/>
+        </geometry>
+        <material name="grey"/>
+      </visual>
+      <collision>
+        <origin xyz="0.0011 -0.0001 0.0194" rpy="0 0 0"/>
+        <geometry>
+          <mesh filename="${meshes_file_direction}/pieces_CoM/link0_CoM.stl" scale="0.001 0.001 0.001"/>
+        </geometry>
+      </collision>
+      <inertial>
+        <origin xyz="0.00011 -0.001 0.0194" />
+        <mass value="8.2e-02" />
+        <inertia ixx="18.5495e-06" ixy="-0.1704e-06" ixz="0.3415e-06"
+                 iyy="29.4750e-06" iyz="0.0015e-06"
+                 izz="23.0866e-06" />
+      </inertial>
+    </link>
+    <joint name="${prefix}joint1" type="revolute">
+      <parent link="${prefix}link0"/>
+      <child link="${prefix}link1"/>
+      <origin xyz="0.012 0 0.036" rpy="${ic_joints[0]} 0  0"/>
+      <axis xyz="0 0 1"/>
+      <limit velocity="4.8" effort="4.1" lower="${-3.14}" upper="${3.14}" />
+      <dynamics damping="0.1"/>
+    </joint>
     <link name="${prefix}link1">
       <visual>
-        <origin xyz="0 0 0" rpy="0 0 0"/>
-        <geometry>
-          <mesh filename="${meshes_file_direction}/link1.stl" scale="0.001 0.001 0.001"/>
-        </geometry>
-        <material name="grey"/>
-      </visual>
-      <collision>
-        <origin xyz="0 0 0" rpy="0 0 0"/>
-        <geometry>
-          <mesh filename="${meshes_file_direction}/link1.stl" scale="0.001 0.001 0.001"/>
+        <origin xyz="0 0.0 0.0277" rpy="1.578 0 0"/>
+        <geometry>
+          <mesh filename="${meshes_file_direction}/pieces_CoM/link1_CoM.stl" scale="0.001 0.001 0.001"/>
+        </geometry>
+        <material name="grey"/>
+      </visual>
+      <collision>
+        <origin xyz="0 0.0 0.0277" rpy="1.578 0 0"/>
+        <geometry>
+          <mesh filename="${meshes_file_direction}/pieces_CoM/link1_CoM.stl" scale="0.001 0.001 0.001"/>
         </geometry>
       </collision>
        <inertial>
-        <origin xyz="3.0876154e-04 0.0000000e+00 -1.2176461e-04" />
-        <mass value="7.9119962e-02" />
-        <inertia ixx="1.2505234e-05" ixy="0.0" ixz="-1.7855208e-07"
-                 iyy="2.1898364e-05" iyz="0.0"
-                 izz="1.9267361e-05" />
-      </inertial>
-    </link>
-    <joint name="${prefix}joint1" type="revolute">
+        <origin xyz="0 0 0.0277 "/>
+        <mass value="10.5e-02" />
+        <inertia ixx="45.0914e-06" ixy="-0.1136e-06" ixz="-0.0084e-06"
+                 iyy="23.7269e-06" iyz="-0.2222e-06"
+                 izz="35.9688e-06" />
+      </inertial>
+    </link>
+    <joint name="${prefix}joint2" type="revolute">
       <parent link="${prefix}link1"/>
       <child link="${prefix}link2"/>
-      <origin xyz="0.012 0.0 0.017" rpy="${ic_joints[0]} 0  0"/>
-      <axis xyz="0 0 1"/>
-      <limit velocity="4.8" effort="1" lower="${-pi}" upper="${pi}" />
+      <origin xyz="0 0.0 0.0433" rpy="1.578 ${ic_joints[1]} 0"/>
+       <axis xyz="0 0 1"/>
+      <limit velocity="4.8" effort="4.1" lower="${-3.14}" upper="${3.14}" />
       <dynamics damping="0.1"/>
     </joint>
     <link name="${prefix}link2">
       <visual>
-        <origin xyz="0 0 0.019" rpy="0 0 0"/>
-        <geometry>
-          <mesh filename="${meshes_file_direction}/link2.stl" scale="0.001 0.001 0.001"/>
-        </geometry>
-        <material name="grey"/>
-      </visual>
-      <collision>
-        <origin xyz="0 0 0.019" rpy="0 0 0"/>
-        <geometry>
-          <mesh filename="${meshes_file_direction}/link2.stl" scale="0.001 0.001 0.001"/>
+        <origin xyz="0.0924 0.0106 0.0003" rpy="0 0 0"/>
+        <geometry>
+          <mesh filename="${meshes_file_direction}/pieces_CoM/link2_CoM.stl" scale="0.001 0.001 0.001"/>
+        </geometry>
+        <material name="grey"/>
+      </visual>
+      <collision>
+        <origin xyz="0.0924 0.0106 0.0003" rpy="0 0 0"/>
+        <geometry>
+          <mesh filename="${meshes_file_direction}/pieces_CoM/link2_CoM.stl" scale="0.001 0.001 0.001"/>
         </geometry>
       </collision>
        <inertial>
-        <origin xyz="-3.0184870e-04 5.4043684e-04 ${0.018 + 2.9433464e-02}" />
-        <mass value="9.8406837e-02" />
-        <inertia ixx="3.4543422e-05" ixy="-1.6031095e-08" ixz="-3.8375155e-07"
-                 iyy="3.2689329e-05" iyz="2.8511935e-08"
-                 izz="1.8850320e-05" />
-      </inertial>
-    </link>
-    <joint name="${prefix}joint2" type="revolute">
+         <origin xyz="0.0924 0.0106 0.0003" />
+        <mass value="14.2e-02" />
+        <inertia ixx="36.9717e-06" ixy="-7.5128e-06" ixz="0.7972e-06"
+                 iyy="236.0399e-06" iyz="0.1582e-06"
+                 izz="233.5145e-06" />
+      </inertial>
+    </link>
+    <joint name="${prefix}joint3" type="revolute">
       <parent link="${prefix}link2"/>
       <child link="${prefix}link3"/>
-      <origin xyz="0.0 0.0 0.0595" rpy="0 ${ic_joints[1]} 0"/>
-      <axis xyz="0 1 0"/>
-      <limit velocity="4.8" effort="1" lower="${-1.5}" upper="${1.5}" />
+      <origin xyz="0.1317 0 0" rpy="0 ${ic_joints[2]} 0"/>
+      <axis xyz="0 0 1"/>
+      <limit velocity="4.8" effort="4.1" lower="${-3.14}" upper="${3.14}" />
       <dynamics damping="0.1"/>
     </joint>
     <link name="${prefix}link3">
       <visual>
-        <origin xyz="0 0 0" rpy="0 0 0"/>
-        <geometry>
-          <mesh filename="${meshes_file_direction}/link3.stl" scale="0.001 0.001 0.001"/>
-        </geometry>
-        <material name="grey"/>
-      </visual>
-      <collision>
-        <origin xyz="0 0 0" rpy="0 0 0"/>
-        <geometry>
-          <mesh filename="${meshes_file_direction}/link3.stl" scale="0.001 0.001 0.001"/>
+        <origin xyz="0.0816 0 0" rpy="0 0 0"/>
+        <geometry>
+          <mesh filename="${meshes_file_direction}/pieces_CoM/link3_CoM.stl" scale="0.001 0.001 0.001"/>
+        </geometry>
+        <material name="grey"/>
+      </visual>
+      <collision>
+        <origin xyz="0.0816 0 0" rpy="0 0 0"/>
+        <geometry>
+          <mesh filename="${meshes_file_direction}/pieces_CoM/link3_CoM.stl" scale="0.001 0.001 0.001"/>
         </geometry>
       </collision>
        <inertial>
-        <origin xyz="1.0308393e-02 3.7743363e-04 1.0170197e-01" />
-        <mass value="1.3850917e-01" />
-        <inertia ixx="3.3055381e-04" ixy="-9.7940978e-08" ixz="-3.8505711e-05"
-                 iyy="3.4290447e-04" iyz="-1.5717516e-06"
-                 izz="6.0346498e-05" />
-      </inertial>
-    </link>
-    <joint name="${prefix}joint3" type="revolute">
+         <origin xyz="0.0816 0 0" />
+        <mass value="13.5e-02" />
+        <inertia ixx="26.8442e-06" ixy="-0.3549e-06" ixz="0.5156e-06"
+                 iyy="193.8335e-06" iyz="0.0095e-06"
+                 izz="181.4661e-06" />
+      </inertial>
+    </link>
+    <joint name="${prefix}joint4" type="revolute">
       <parent link="${prefix}link3"/>
       <child link="${prefix}link4"/>
-      <origin xyz="0.024 0 0.128" rpy="0 ${ic_joints[2]} 0"/>
-      <axis xyz="0 1 0"/>
-      <limit velocity="4.8" effort="1" lower="${-1.5}" upper="${1.4}" />
+      <origin xyz="0.1253 0.0 0.0" rpy="0 ${ic_joints[3]} 0"/>
+      <axis xyz="0 0 1"/>
+       <!--
+      <limit velocity="4.8" effort="4.1" lower="${-3.14}" upper="${3.14}" />
+      -->
+      <limit velocity="4.8" effort="4.1" lower="${-3.14}" upper="${3.14}" />
       <dynamics damping="0.1"/>
     </joint>
     <link name="${prefix}link4">
       <visual>
-        <origin xyz="0 0 0" rpy="0 0 0"/>
-        <geometry>
-          <mesh filename="${meshes_file_direction}/link4.stl" scale="0.001 0.001 0.001"/>
-        </geometry>
-        <material name="grey"/>
-      </visual>
-      <collision>
-        <origin xyz="0 0 0" rpy="0 0 0"/>
-        <geometry>
-          <mesh filename="${meshes_file_direction}/link4.stl" scale="0.001 0.001 0.001"/>
-        </geometry>
-      </collision>
-       <inertial>
-        <origin xyz="9.0909590e-02 3.8929816e-04 2.2413279e-04" />
-        <mass value="1.3274562e-01" />
-        <inertia ixx="3.0654178e-05" ixy="-1.2764155e-06" ixz="-2.6874417e-07"
-                 iyy="2.4230292e-04" iyz="1.1559550e-08"
-                 izz="2.5155057e-04" />
-      </inertial>
-    </link>
-    <joint name="${prefix}joint4" type="revolute">
+        <origin xyz="0.0415 -0.00574 0" rpy="1.57 0 0"/>
+        <geometry>
+          <mesh filename="${meshes_file_direction}/pieces_CoM/link4_CoM.stl" scale="0.001 0.001 0.001"/>
+        </geometry>
+        <material name="grey"/>
+      </visual>
+      <collision>
+        <origin xyz="0.0702 0.0035 0" rpy="0 0 0"/>
+        <geometry>
+          <mesh filename="${meshes_file_direction}/pieces_CoM/link4_CoM.stl" scale="0.001 0.001 0.001"/>
+        </geometry>
+      </collision>
+      <inertial>
+        <origin xyz="0.0702 0.0035 0" />
+        <mass value="23.6e-02" />
+        <inertia ixx="237.6911e-06" ixy="20.1638e-06" ixz="-0.0052e-06"
+                 iyy="363.9779e-06" iyz="0.0704e-06"
+                 izz="243.4494e-06" />
+      </inertial>
+    </link>
+    <joint name="${prefix}gripper_left_joint" type="prismatic">
       <parent link="${prefix}link4"/>
-      <child link="${prefix}link5"/>
-      <origin xyz="0.124 0.0 0.0" rpy="0 0 0"/>
-      <origin xyz="0.124 0.0 0.0" rpy="0 ${ic_joints[3]} 0"/>
-      <axis xyz="0 1 0"/>
-      <limit velocity="4.8" effort="1" lower="${-1.7}" upper="${1.97}" />
-      <dynamics damping="0.1"/>
-    </joint>
-    <link name="${prefix}link5">
-      <visual>
-        <origin xyz="0 0 0" rpy="0 0 0"/>
-        <geometry>
-          <mesh filename="${meshes_file_direction}/link5.stl" scale="0.001 0.001 0.001"/>
-        </geometry>
-        <material name="grey"/>
-      </visual>
-      <collision>
-        <origin xyz="0 0 0" rpy="0 0 0"/>
-        <geometry>
-          <mesh filename="${meshes_file_direction}/link5.stl" scale="0.001 0.001 0.001"/>
-        </geometry>
-      </collision>
-       <inertial>
-        <origin xyz="4.4206755e-02 3.6839985e-07 8.9142216e-03" />
-        <mass value="1.4327573e-01" />
-        <inertia ixx="8.0870749e-05" ixy="0.0" ixz="-1.0157896e-06"
-                 iyy="7.5980465e-05" iyz="0.0"
-                 izz="9.3127351e-05" />
-      </inertial>
-    </link>
-    <joint name="${prefix}gripper_left_joint" type="prismatic">
-      <parent link="${prefix}link5"/>
       <child link="${prefix}gripper_left_link"/>
-      <origin xyz="0.0817 0.021 0.0" rpy="0 0 0"/>
-      <axis xyz="0 1 0"/>
-      <limit velocity="4.8" effort="1" lower="-0.010" upper="0.019" />
+      <origin rpy="-1.56 0 -1.56" xyz="0.0665 0 0"/>
+      <axis xyz="0 0 1"/>
+      <limit velocity="4.8" effort="4.1" lower="${-3.14}" upper="${3.14}" />
       <dynamics damping="0.1"/>
     </joint>
     <link name="${prefix}gripper_left_link">
       <visual>
-        <origin xyz="0 0 0" rpy="0 0 0"/>
-        <geometry>
-          <mesh filename="${meshes_file_direction}/gripper_left_palm.stl" scale="0.001 0.001 0.001"/>
-        </geometry>
-        <material name="grey"/>
-      </visual>
-      <collision>
-        <origin xyz="0 0 0" rpy="0 0 0"/>
-        <geometry>
-          <mesh filename="${meshes_file_direction}/gripper_left_palm.stl" scale="0.001 0.001 0.001"/>
-        </geometry>
-      </collision>
-      <inertial>
-        <origin xyz="0 0 0" />
-        <mass value="1.0e-03" />
-        <inertia ixx="1.0e-06" ixy="0.0" ixz="0.0"
-                 iyy="1.0e-06" iyz="0.0"
-                 izz="1.0e-06" />
+        <origin xyz="0 0.0452 0.0274" rpy="0 -1.57 0"/>
+        <geometry>
+          <mesh filename="${meshes_file_direction}/pieces_CoM/gripper_left_palm_CoM.stl" scale="0.001 0.001 0.001"/>
+        </geometry>
+        <material name="grey"/>
+      </visual>
+      <collision>
+        <origin xyz="0 0.0452 0.0274" rpy="0 -1.57 0"/>
+        <geometry>
+          <mesh filename="${meshes_file_direction}/pieces_CoM/gripper_left_palm_CoM.stl" scale="0.001 0.001 0.001"/>
+        </geometry>
+      </collision>
+      <inertial>
+        <origin xyz="0 0.0452 0.0274" rpy="0 -1.57 0"/>
+        <mass value="1.0e-06" />
+        <inertia ixx="1.0e-12" ixy="0.0" ixz="0.0"
+                 iyy="1.0e-12" iyz="0.0"
+                 izz="1.0e-12" />
       </inertial>
     </link>
@@ -185,9 +188,9 @@
     <link name="dummy_mimic_fix"/>
     <joint name="${prefix}gripper_right_joint" type="prismatic">
-      <parent link="${prefix}link5"/>
+      <parent link="${prefix}link4"/>
       <child link="${prefix}gripper_right_link"/>
-      <origin xyz="0.0817 -0.021 0" rpy="0 0 0"/>
-      <axis xyz="0 -1 0"/>
-      <limit velocity="4.8" effort="1" lower="-0.010" upper="0.019" />
+      <origin rpy="-1.56 0 -1.56" xyz="0.0665 0 0"/>
+      <axis xyz="0 0 1"/>
+      <limit velocity="4.8" effort="4.1" lower="${-3.14}" upper="${3.14}" />
       <mimic joint="${prefix}gripper_left_joint" multiplier="1"/>
       <dynamics damping="0.1"/>
@@ -195,26 +198,26 @@
     <link name="${prefix}gripper_right_link">
       <visual>
-        <origin xyz="0 0 0" rpy="0 0 0"/>
-        <geometry>
-          <mesh filename="${meshes_file_direction}/gripper_right_palm.stl" scale="0.001 0.001 0.001"/>
-        </geometry>
-        <material name="grey"/>
-      </visual>
-      <collision>
-        <origin xyz="0 0 0" rpy="0 0 0"/>
-        <geometry>
-          <mesh filename="${meshes_file_direction}/gripper_right_palm.stl" scale="0.001 0.001 0.001"/>
-        </geometry>
-      </collision>
-      <inertial>
-        <origin xyz="0 0 0" />
-        <mass value="1.0e-03" />
-        <inertia ixx="1.0e-06" ixy="0.0" ixz="0.0"
-                 iyy="1.0e-06" iyz="0.0"
-                 izz="1.0e-06" />
+        <origin xyz="0 -0.0452 0.0274" rpy="0 -1.57 0"/>
+        <geometry>
+          <mesh filename="${meshes_file_direction}/pieces_CoM/gripper_right_palm_CoM.stl" scale="0.001 0.001 0.001"/>
+        </geometry>
+        <material name="grey"/>
+      </visual>
+      <collision>
+        <origin xyz="0 -0.0452 0.0274" rpy="0 -1.57 0"/>
+        <geometry>
+          <mesh filename="${meshes_file_direction}/pieces_CoM/gripper_right_palm_CoM.stl" scale="0.001 0.001 0.001"/>
+        </geometry>
+      </collision>
+      <inertial>
+        <origin xyz="0 0.0452 0.0274" rpy="0 -1.57 0"/>
+        <mass value="1.0e-06" />
+        <inertia ixx="1.0e-12" ixy="0.0" ixz="0.0"
+                 iyy="1.0e-12" iyz="0.0"
+                 izz="1.0e-12" />
       </inertial>
     </link>
     <joint name="${prefix}end_effector_joint" type="fixed">
-      <parent link="${prefix}link5"/>
+      <parent link="${prefix}link4"/>
       <child link="${prefix}end_effector_link"/>
       <origin xyz="0.126 0.0 0.0" rpy="0 0 0"/>

File: open_manipulator_x_description/urdf/open_manipulator_x_robot.urdf.xacro (robot description, xacro)
@@ -33,5 +33,5 @@
     <origin xyz="0 0 0" rpy="0 0 0"/>
     <parent link="world"/>
-    <child link="$(arg prefix)link1"/>
+    <child link="$(arg prefix)link0"/>
   </joint>
 </robot>
