Commit message: feat(IC): implement initial conditions on arm joints

File: open_manipulator_x_description/urdf/open_manipulator_x.urdf.xacro (robot description, xacro)
@@ -1,5 +1,6 @@
 <?xml version="1.0"?>
 <robot xmlns:xacro="http://www.ros.org/wiki/xacro">
-  <xacro:macro name="open_manipulator_x" params="prefix=''">
+  <xacro:macro name="open_manipulator_x" params="prefix:=''
+    ic_joints:=${[0.0, 0.0, 0.0, 0.0]}">
     <xacro:property
       name="meshes_file_direction"
@@ -30,5 +31,5 @@
       <parent link="${prefix}link1"/>
       <child link="${prefix}link2"/>
-      <origin xyz="0.012 0.0 0.017" rpy="0 0 0"/>
+      <origin xyz="0.012 0.0 0.017" rpy="${ic_joints[0]} 0  0"/>
       <axis xyz="0 0 1"/>
       <limit velocity="4.8" effort="1" lower="${-pi}" upper="${pi}" />
@@ -60,5 +61,5 @@
       <parent link="${prefix}link2"/>
       <child link="${prefix}link3"/>
-      <origin xyz="0.0 0.0 0.0595" rpy="0 0 0"/>
+      <origin xyz="0.0 0.0 0.0595" rpy="0 ${ic_joints[1]} 0"/>
       <axis xyz="0 1 0"/>
       <limit velocity="4.8" effort="1" lower="${-1.5}" upper="${1.5}" />
@@ -90,5 +91,5 @@
       <parent link="${prefix}link3"/>
       <child link="${prefix}link4"/>
-      <origin xyz="0.024 0 0.128" rpy="0 0 0"/>
+      <origin xyz="0.024 0 0.128" rpy="0 ${ic_joints[2]} 0"/>
       <axis xyz="0 1 0"/>
       <limit velocity="4.8" effort="1" lower="${-1.5}" upper="${1.4}" />
@@ -121,4 +122,5 @@
       <child link="${prefix}link5"/>
       <origin xyz="0.124 0.0 0.0" rpy="0 0 0"/>
+      <origin xyz="0.124 0.0 0.0" rpy="0 ${ic_joints[3]} 0"/>
       <axis xyz="0 1 0"/>
       <limit velocity="4.8" effort="1" lower="${-1.7}" upper="${1.97}" />

File: open_manipulator_x_description/urdf/open_manipulator_x_robot.urdf.xacro (robot description, xacro)
@@ -7,4 +7,5 @@
   <xacro:arg name="fake_sensor_commands" default="false" />
   <xacro:arg name="port_name" default="/dev/ttyUSB0" />
+  <xacro:arg name="ic_joints" default="[0.0, 0.0, 0.0, 0.0]"/>
   <!-- Import Rviz colors -->
   <xacro:include filename="$(find open_manipulator_x_description)/gazebo/materials.xacro" />
@@ -12,7 +13,7 @@
   <xacro:include filename="$(find open_manipulator_x_description)/gazebo/open_manipulator_x.gazebo.xacro" />
   <!-- Import URDF -->
-  <xacro:include filename="$(find open_manipulator_x_description)/urdf/open_manipulator_x.urdf.xacro" />
+  <xacro:include filename="$(find open_manipulator_x_description)/urdf/open_manipulator_x.urdf.xacro"/>
   <xacro:include filename="$(find open_manipulator_x_description)/ros2_control/open_manipulator_x_system.ros2_control.xacro" />
-  <xacro:open_manipulator_x prefix="$(arg prefix)" />
+  <xacro:open_manipulator_x prefix="$(arg prefix)" ic_joints="${list($(arg ic_joints))}"/>
   <xacro:open_manipulator_x_gazebo prefix="$(arg prefix)" />
   <xacro:open_manipulator_x_system

Commit message: fix(sdf): wrong EE pose of collision and inertia

File: open_manipulator_x_description/urdf/open_manipulator_x.urdf.xacro (robot description, xacro)
@@ -139,5 +139,5 @@
       </visual>
       <collision>
-        <origin xyz="0.0702 0.0035 0" rpy="0 0 0"/>
+        <origin xyz="0.0415 -0.00574 0" rpy="1.57 0 0"/>
         <geometry>
           <mesh filename="${meshes_file_direction}/pieces_CoM/link4_CoM.stl" scale="0.001 0.001 0.001"/>
@@ -145,5 +145,5 @@
       </collision>
       <inertial>
-        <origin xyz="0.0702 0.0035 0" />
+        <origin xyz="0.0415 -0.00574 0" rpy="1.57 0 0" />
         <mass value="23.6e-02" />
         <inertia ixx="237.6911e-06" ixy="20.1638e-06" ixz="-0.0052e-06"
@@ -211,5 +211,5 @@
       </collision>
       <inertial>
-        <origin xyz="0 0.0452 0.0274" rpy="0 -1.57 0"/>
+        <origin xyz="0 -0.0452 0.0274" rpy="0 -1.57 0"/>
         <mass value="1.0e-06" />
         <inertia ixx="1.0e-12" ixy="0.0" ixz="0.0"

Commit message: fix(CoM): wrong CoM on EE

File: open_manipulator_x_description/urdf/open_manipulator_x.urdf.xacro (robot description, xacro)
@@ -144,6 +144,7 @@
         </geometry>
       </collision>
-      <inertial>
-        <origin xyz="0.0415 -0.00574 0" rpy="1.57 0 0" />
+      <!-- TODO Compute again the inertia matrix as 3 difference pieces and not like a unique piece-->
+      <inertial>
+        <origin xyz="0.0702 0.0035 0" />
         <mass value="23.6e-02" />
         <inertia ixx="237.6911e-06" ixy="20.1638e-06" ixz="-0.0052e-06"
